File: desk_clock/board/Desk Clock.brd (EAGLE design)
At the start: 94.6 x 43.8 mm, 14 parts, among them IC1 PIC16F628P, IC2 MAX7219CNG, U1 TMP75D, X1 22-23-2021

Commit message: HW revision 1.1. Added a 0.1uF capacitor to improve electric stability and reduce drifting. Also removed version number from the pcb filenames (it's embedded in the schematic and pcb layout now). Firmware has been updated to deal with the random auto-halt of the DS1302 module in software, and the polling/refresh rate of the clock has been reduced by adding a delay in the loop. Some NOPs were removed from the DS1302 communication routines as they were not really needed due to the low frequency at which the PIC is running.
Parts:
- added C2: 0.1uF, rcl:C025-025X050
- moved C1 2.62 mm to (47.6, 14.0)
Connections:
- net GND: now also C2.2
- net VDD: now also C2.1
Routing:
- net VDD: track 155.7 -> 154.8 mm
Other:
- board text added: "DESK CLOCK v1.1"
Changed lines of the file:
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@@
 <hole x="20" y="4.635" drill="3"/>
 <hole x="3" y="41.635" drill="3"/>
+<text x="3.81" y="37.465" size="1.778" layer="16" rot="MR270">DESK CLOCK v1.1</text>
 </plain>
 <attributes>
@@
 <attribute name="MPN" value="22-23-2021" x="7.62" y="13.335" size="1.778" layer="27" display="off"/>
 </element>
-<element name="C1" library="rcl" package="E2-4" value="10uF" x="46.99" y="16.51" rot="R180"/>
+<element name="C1" library="rcl" package="E2-4" value="10uF" x="47.625" y="13.97" rot="R180"/>
+<element name="C2" library="rcl" package="C025-025X050" value="0.1uF" x="47.625" y="17.78" rot="R180"/>
 </elements>
 <signals>
@@
 <wire x1="40.64" y1="27.305" x2="44.45" y2="27.305" width="0.6096" layer="16"/>
 <wire x1="44.45" y1="27.305" x2="48.895" y2="22.86" width="0.6096" layer="16"/>
-<wire x1="48.895" y1="22.86" x2="48.895" y2="16.51" width="0.6096" layer="16"/>
-<wire x1="48.895" y1="16.51" x2="48.895" y2="14.605" width="0.6096" layer="16"/>
-<wire x1="48.895" y1="14.605" x2="51.435" y2="12.065" width="0.6096" layer="16"/>
-<wire x1="51.435" y1="12.065" x2="51.435" y2="8.89" width="0.6096" layer="16"/>
+<wire x1="51.435" y1="11.43" x2="51.435" y2="8.89" width="0.6096" layer="16"/>
 <contactref element="X1" pad="1"/>
 <wire x1="6.62" y1="14.24" x2="6.35" y2="13.335" width="0.6096" layer="16"/>
@@
 <wire x1="60.325" y1="4.445" x2="55.88" y2="4.445" width="0.6096" layer="16"/>
 <contactref element="C1" pad="+"/>
-<wire x1="48.006" y1="16.51" x2="48.895" y2="16.51" width="0.6096" layer="16"/>
 <wire x1="60.325" y1="4.445" x2="60.96" y2="5.08" width="0.6096" layer="16"/>
 <wire x1="60.96" y1="5.08" x2="60.96" y2="8.89" width="0.6096" layer="16"/>
@@
 <wire x1="71.12" y1="11.43" x2="69.85" y2="12.7" width="0.6096" layer="16"/>
 <wire x1="69.85" y1="12.7" x2="69.85" y2="14.605" width="0.6096" layer="16"/>
+<contactref element="C2" pad="1"/>
+<wire x1="48.895" y1="22.86" x2="48.895" y2="17.78" width="0.6096" layer="16"/>
+<wire x1="48.895" y1="17.78" x2="48.895" y2="13.97" width="0.6096" layer="16"/>
+<wire x1="48.895" y1="13.97" x2="48.641" y2="13.97" width="0" layer="19" extent="1-16"/>
+<wire x1="48.895" y1="13.97" x2="51.435" y2="11.43" width="0.6096" layer="16"/>
 </signal>
 <signal name="N$1">
@@
 <wire x1="17.145" y1="19.685" x2="17.145" y2="31.055" width="0.6096" layer="16"/>
 <wire x1="17.145" y1="31.055" x2="17.78" y2="31.69" width="0.6096" layer="16"/>
-<wire x1="48.895" y1="11.176" x2="48.895" y2="5.715" width="0.6096" layer="16"/>
+<wire x1="48.895" y1="10.541" x2="48.895" y2="5.715" width="0.6096" layer="16"/>
 <contactref element="C1" pad="-"/>
-<wire x1="48.895" y1="11.176" x2="45.974" y2="14.097" width="0.6096" layer="16"/>
-<wire x1="45.974" y1="16.51" x2="45.72" y2="16.764" width="0.6096" layer="16"/>
-<wire x1="45.72" y1="16.764" x2="45.72" y2="23.495" width="0.6096" layer="16"/>
-<wire x1="45.72" y1="23.495" x2="43.18" y2="26.035" width="0.6096" layer="16"/>
+<wire x1="46.355" y1="22.86" x2="43.18" y2="26.035" width="0.6096" layer="16"/>
 <wire x1="35.56" y1="26.035" x2="34.29" y2="27.305" width="0.6096" layer="16"/>
 <wire x1="34.29" y1="27.305" x2="33.02" y2="27.305" width="0.6096" layer="16"/>
-<wire x1="45.974" y1="14.097" x2="45.974" y2="16.51" width="0.6096" layer="16"/>
 <wire x1="35.56" y1="26.035" x2="43.18" y2="26.035" width="0.6096" layer="16"/>
+<contactref element="C2" pad="2"/>
+<wire x1="46.355" y1="22.86" x2="46.355" y2="17.78" width="0.6096" layer="16"/>
+<wire x1="46.355" y1="17.78" x2="46.355" y2="14.224" width="0.6096" layer="16"/>
+<wire x1="46.355" y1="14.224" x2="46.609" y2="13.97" width="0.6096" layer="16"/>
+<wire x1="46.609" y1="13.97" x2="46.609" y2="12.827" width="0.6096" layer="16"/>
+<wire x1="46.609" y1="12.827" x2="48.895" y2="10.541" width="0.6096" layer="16"/>
 </signal>
 <signal name="N$19">
